Commit message: For the time being

File: quarobo_description/robots/quarobo.urdf.xacro (robot description, xacro)
@@ -9,4 +9,9 @@
     </joint>
     <link name="body_link">
+        <inertial>
+            <origin xyz="0 0 0" rpy="0 0 0"/>
+            <mass value="0.02"/>
+            <inertia ixx="0.1" ixy="0" ixz="0" iyy="0.1" iyz="0" izz="0.1"   />
+        </inertial>
         <visual>
             <geometry>
@@ -16,72 +21,78 @@
             <material name="pink"/>
         </visual>
-    </link>
-    <!-- === Front right === -->
-    <xacro:leg_macro prefix="FRS" parent="body_link" type="revolute" mesh="front_Shoulder_R.stl" color="green">
-        <axis xyz="0 1 0"/>
-        <origin xyz="-0.027 -0.04905 -0.00075" rpy="0 0 0"/>
-    </xacro:leg_macro>
-    <xacro:leg_macro prefix="FRL" parent="FRS_link" type="revolute" mesh="front_Leg_R.stl" color="blue">
-        <axis xyz="1 0 0"/>
-        <origin xyz="0 -0.022304 -0.01230" rpy="1.57 0 0"/>
-    </xacro:leg_macro>
-    <xacro:leg_macro prefix="FRF" parent="FRL_link" type="revolute" mesh="front_Foot_R.stl" color="purple">
-        <axis xyz="1 0 0"/>
-        <origin xyz="-0.015546 -0.054 0" rpy="0 0 0"/>
-    </xacro:leg_macro>
-    <xacro:leg_macro prefix="FRT" parent="FRF_link" type="fixed" mesh="front_Toes_R.stl" color="orange">
-        <axis xyz="1 0 0"/>
-        <origin xyz="-0.003 -0.088 0" rpy="0 0 0"/>
-    </xacro:leg_macro>
-    <!-- === Front left === -->
-    <xacro:leg_macro prefix="FLS" parent="body_link" type="revolute" mesh="front_Shoulder_L.stl" color="green">
-        <axis xyz="0 1 0"/>
-        <origin xyz="0.027 -0.04905 -0.00075" rpy="0 0 0"/>
-    </xacro:leg_macro>
-    <xacro:leg_macro prefix="FLL" parent="FLS_link" type="revolute" mesh="front_Leg_L.stl" color="blue">
-        <axis xyz="1 0 0"/>
-        <origin xyz="0 -0.022304 -0.01230" rpy="1.57 0 0"/>
-    </xacro:leg_macro>
-    <xacro:leg_macro prefix="FLF" parent="FLL_link" type="revolute" mesh="front_Foot_L.stl" color="purple">
-        <axis xyz="1 0 0"/>
-        <origin xyz="0.015546 -0.054 0" rpy="0 0 0"/>
-    </xacro:leg_macro>
-    <xacro:leg_macro prefix="FLT" parent="FLF_link" type="fixed" mesh="front_Toes_L.stl" color="orange">
-        <axis xyz="1 0 0"/>
-        <origin xyz="0.003 -0.088 0" rpy="0 0 0"/>
-    </xacro:leg_macro>
-    <!-- === Rear right === -->
-    <xacro:leg_macro prefix="RRS" parent="body_link" type="revolute" mesh="rear_Shoulder_R.stl" color="green">
-        <axis xyz="0 1 0"/>
-        <origin xyz="-0.027 0.04905 -0.00075" rpy="0 0 0"/>
-    </xacro:leg_macro>
-    <xacro:leg_macro prefix="RRL" parent="RRS_link" type="revolute" mesh="rear_Leg_R.stl" color="blue">
-        <axis xyz="1 0 0"/>
-        <origin xyz="0 0.022304 -0.01230" rpy="-1.57 0 0"/>
-    </xacro:leg_macro>
-    <xacro:leg_macro prefix="RRF" parent="RRL_link" type="revolute" mesh="rear_Foot_R.stl" color="purple">
-        <axis xyz="1 0 0"/>
-        <origin xyz="-0.015546 0.054 0" rpy="0 0 0"/>
-    </xacro:leg_macro>
-    <xacro:leg_macro prefix="RRT" parent="RRF_link" type="fixed" mesh="rear_Toes_R.stl" color="orange">
-        <axis xyz="1 0 0"/>
-        <origin xyz="-0.003 0.088 0" rpy="0 0 0"/>
-    </xacro:leg_macro>
-    <!-- === Rear left === -->
-    <xacro:leg_macro prefix="RLS" parent="body_link" type="revolute" mesh="rear_Shoulder_L.stl" color="green">
-        <axis xyz="0 1 0"/>
-        <origin xyz="0.027 0.04905 -0.00075" rpy="0 0 0"/>
-    </xacro:leg_macro>
-    <xacro:leg_macro prefix="RLL" parent="RLS_link" type="revolute" mesh="rear_Leg_L.stl" color="blue">
-        <axis xyz="1 0 0"/>
-        <origin xyz="0 0.022304 -0.01230" rpy="-1.57 0 0"/>
-    </xacro:leg_macro>
-    <xacro:leg_macro prefix="RLF" parent="RLL_link" type="revolute" mesh="rear_Foot_L.stl" color="purple">
-        <axis xyz="1 0 0"/>
-        <origin xyz="0.015546 0.054 0" rpy="0 0 0"/>
-    </xacro:leg_macro>
-    <xacro:leg_macro prefix="RLT" parent="RLF_link" type="fixed" mesh="rear_Toes_L.stl" color="orange">
-        <axis xyz="1 0 0"/>
-        <origin xyz="0.003 0.088 0" rpy="0 0 0"/>
-    </xacro:leg_macro>
-</robot>
+        <collision>
+            <origin xyz="0 0 0" rpy="0 0 0"/>
+            <geometry>
+                <box size="0.07160 0.09810 0.01960"/>
+            </geometry>
+        </collision>
+        </link>
+        <!-- === Front right === -->
+        <xacro:leg_macro prefix="FRS" parent="body_link" type="revolute" mesh="front_Shoulder_R.stl" color="green">
+            <axis xyz="0 1 0"/>
+            <origin xyz="-0.027 -0.04905 -0.00075" rpy="0 0 0"/>
+        </xacro:leg_macro>
+        <xacro:leg_macro prefix="FRL" parent="FRS_link" type="revolute" mesh="front_Leg_R.stl" color="blue">
+            <axis xyz="1 0 0"/>
+            <origin xyz="0 -0.022304 -0.01230" rpy="1.57 0 0"/>
+        </xacro:leg_macro>
+        <xacro:leg_macro prefix="FRF" parent="FRL_link" type="revolute" mesh="front_Foot_R.stl" color="purple">
+            <axis xyz="1 0 0"/>
+            <origin xyz="-0.015546 -0.054 0" rpy="0 0 0"/>
+        </xacro:leg_macro>
+        <xacro:leg_macro prefix="FRT" parent="FRF_link" type="fixed" mesh="front_Toes_R.stl" color="orange">
+            <axis xyz="1 0 0"/>
+            <origin xyz="-0.003 -0.088 0" rpy="0 0 0"/>
+        </xacro:leg_macro>
+        <!-- === Front left === -->
+        <xacro:leg_macro prefix="FLS" parent="body_link" type="revolute" mesh="front_Shoulder_L.stl" color="green">
+            <axis xyz="0 1 0"/>
+            <origin xyz="0.027 -0.04905 -0.00075" rpy="0 0 0"/>
+        </xacro:leg_macro>
+        <xacro:leg_macro prefix="FLL" parent="FLS_link" type="revolute" mesh="front_Leg_L.stl" color="blue">
+            <axis xyz="1 0 0"/>
+            <origin xyz="0 -0.022304 -0.01230" rpy="1.57 0 0"/>
+        </xacro:leg_macro>
+        <xacro:leg_macro prefix="FLF" parent="FLL_link" type="revolute" mesh="front_Foot_L.stl" color="purple">
+            <axis xyz="1 0 0"/>
+            <origin xyz="0.015546 -0.054 0" rpy="0 0 0"/>
+        </xacro:leg_macro>
+        <xacro:leg_macro prefix="FLT" parent="FLF_link" type="fixed" mesh="front_Toes_L.stl" color="orange">
+            <axis xyz="1 0 0"/>
+            <origin xyz="0.003 -0.088 0" rpy="0 0 0"/>
+        </xacro:leg_macro>
+        <!-- === Rear right === -->
+        <xacro:leg_macro prefix="RRS" parent="body_link" type="revolute" mesh="rear_Shoulder_R.stl" color="green">
+            <axis xyz="0 1 0"/>
+            <origin xyz="-0.027 0.04905 -0.00075" rpy="0 0 0"/>
+        </xacro:leg_macro>
+        <xacro:leg_macro prefix="RRL" parent="RRS_link" type="revolute" mesh="rear_Leg_R.stl" color="blue">
+            <axis xyz="1 0 0"/>
+            <origin xyz="0 0.022304 -0.01230" rpy="-1.57 0 0"/>
+        </xacro:leg_macro>
+        <xacro:leg_macro prefix="RRF" parent="RRL_link" type="revolute" mesh="rear_Foot_R.stl" color="purple">
+            <axis xyz="1 0 0"/>
+            <origin xyz="-0.015546 0.054 0" rpy="0 0 0"/>
+        </xacro:leg_macro>
+        <xacro:leg_macro prefix="RRT" parent="RRF_link" type="fixed" mesh="rear_Toes_R.stl" color="orange">
+            <axis xyz="1 0 0"/>
+            <origin xyz="-0.003 0.088 0" rpy="0 0 0"/>
+        </xacro:leg_macro>
+        <!-- === Rear left === -->
+        <xacro:leg_macro prefix="RLS" parent="body_link" type="revolute" mesh="rear_Shoulder_L.stl" color="green">
+            <axis xyz="0 1 0"/>
+            <origin xyz="0.027 0.04905 -0.00075" rpy="0 0 0"/>
+        </xacro:leg_macro>
+        <xacro:leg_macro prefix="RLL" parent="RLS_link" type="revolute" mesh="rear_Leg_L.stl" color="blue">
+            <axis xyz="1 0 0"/>
+            <origin xyz="0 0.022304 -0.01230" rpy="-1.57 0 0"/>
+        </xacro:leg_macro>
+        <xacro:leg_macro prefix="RLF" parent="RLL_link" type="revolute" mesh="rear_Foot_L.stl" color="purple">
+            <axis xyz="1 0 0"/>
+            <origin xyz="0.015546 0.054 0" rpy="0 0 0"/>
+        </xacro:leg_macro>
+        <xacro:leg_macro prefix="RLT" parent="RLF_link" type="fixed" mesh="rear_Toes_L.stl" color="orange">
+            <axis xyz="1 0 0"/>
+            <origin xyz="0.003 0.088 0" rpy="0 0 0"/>
+        </xacro:leg_macro>
+    </robot>

File: quarobo_description/urdf/leg/leg.urdf.xacro (robot description, xacro)
@@ -11,4 +11,9 @@
         </joint>
         <link name="${prefix}_link">
+            <inertial>
+                <origin xyz="0 0 0" rpy="0 0 0"/>
+                <mass value="0.02"/>
+                <inertia ixx="0.1" ixy="0" ixz="0" iyy="0.1" iyz="0" izz="0.1"/>
+            </inertial>
             <visual>
                 <geometry>
@@ -18,4 +23,10 @@
                 <material name="${color}"/>
             </visual>
+            <collision>
+                <origin xyz="0 0 0" rpy="0 0 0"/>
+                <geometry>
+                    <xacro:insert_block name="link_box"/>
+                </geometry>
+            </collision>
         </link>
     </xacro:macro>

Commit message: Update:Gazebo preparation;

File: quarobo_description/robots/quarobo.urdf.xacro (robot description, xacro)
@@ -7,10 +7,11 @@
         <parent link="base_link"/>
         <child link="body_link"/>
+        <origin xyz="0 0 0.16505" rpy="0 0 0"/>
     </joint>
     <link name="body_link">
         <inertial>
             <origin xyz="0 0 0" rpy="0 0 0"/>
-            <mass value="0.02"/>
-            <inertia ixx="0.1" ixy="0" ixz="0" iyy="0.1" iyz="0" izz="0.1"   />
+            <mass value="0.020"/>
+            <inertia ixx="0.1" ixy="0" ixz="0" iyy="0.1" iyz="0" izz="0.1"/>
         </inertial>
         <visual>
@@ -24,24 +25,28 @@
             <origin xyz="0 0 0" rpy="0 0 0"/>
             <geometry>
-                <box size="0.07160 0.09810 0.01960"/>
+                <box size="0.07160 0.09810 0.02410"/>
             </geometry>
         </collision>
-        </link>
+    </link>
         <!-- === Front right === -->
         <xacro:leg_macro prefix="FRS" parent="body_link" type="revolute" mesh="front_Shoulder_R.stl" color="green">
             <axis xyz="0 1 0"/>
             <origin xyz="-0.027 -0.04905 -0.00075" rpy="0 0 0"/>
+            <box size="0.032107 0.031304 0.01960"/>
         </xacro:leg_macro>
         <xacro:leg_macro prefix="FRL" parent="FRS_link" type="revolute" mesh="front_Leg_R.stl" color="blue">
             <axis xyz="1 0 0"/>
             <origin xyz="0 -0.022304 -0.01230" rpy="1.57 0 0"/>
+            <box size="0.02905 0.07160 0.01960"/>
         </xacro:leg_macro>
         <xacro:leg_macro prefix="FRF" parent="FRL_link" type="revolute" mesh="front_Foot_R.stl" color="purple">
             <axis xyz="1 0 0"/>
             <origin xyz="-0.015546 -0.054 0" rpy="0 0 0"/>
+            <box size="0.010 0.099465 0.010"/>
         </xacro:leg_macro>
         <xacro:leg_macro prefix="FRT" parent="FRF_link" type="fixed" mesh="front_Toes_R.stl" color="orange">
             <axis xyz="1 0 0"/>
             <origin xyz="-0.003 -0.088 0" rpy="0 0 0"/>
+            <box size="0.020 0.020 0.020"/>
         </xacro:leg_macro>
         <!-- === Front left === -->
@@ -49,16 +54,20 @@
             <axis xyz="0 1 0"/>
             <origin xyz="0.027 -0.04905 -0.00075" rpy="0 0 0"/>
+            <box size="0.032107 0.031304 0.01960"/>
         </xacro:leg_macro>
         <xacro:leg_macro prefix="FLL" parent="FLS_link" type="revolute" mesh="front_Leg_L.stl" color="blue">
             <axis xyz="1 0 0"/>
             <origin xyz="0 -0.022304 -0.01230" rpy="1.57 0 0"/>
+            <box size="0.02905 0.07160 0.01960"/>
         </xacro:leg_macro>
         <xacro:leg_macro prefix="FLF" parent="FLL_link" type="revolute" mesh="front_Foot_L.stl" color="purple">
             <axis xyz="1 0 0"/>
             <origin xyz="0.015546 -0.054 0" rpy="0 0 0"/>
+            <box size="0.010 0.099465 0.010"/>
         </xacro:leg_macro>
         <xacro:leg_macro prefix="FLT" parent="FLF_link" type="fixed" mesh="front_Toes_L.stl" color="orange">
             <axis xyz="1 0 0"/>
             <origin xyz="0.003 -0.088 0" rpy="0 0 0"/>
+            <box size="0.020 0.020 0.020"/>
         </xacro:leg_macro>
         <!-- === Rear right === -->
@@ -66,16 +75,20 @@
             <axis xyz="0 1 0"/>
             <origin xyz="-0.027 0.04905 -0.00075" rpy="0 0 0"/>
+            <box size="0.032107 0.031304 0.01960"/>
         </xacro:leg_macro>
         <xacro:leg_macro prefix="RRL" parent="RRS_link" type="revolute" mesh="rear_Leg_R.stl" color="blue">
             <axis xyz="1 0 0"/>
             <origin xyz="0 0.022304 -0.01230" rpy="-1.57 0 0"/>
+            <box size="0.02905 0.07160 0.01960"/>
         </xacro:leg_macro>
         <xacro:leg_macro prefix="RRF" parent="RRL_link" type="revolute" mesh="rear_Foot_R.stl" color="purple">
             <axis xyz="1 0 0"/>
             <origin xyz="-0.015546 0.054 0" rpy="0 0 0"/>
+            <box size="0.010 0.099465 0.010"/>
         </xacro:leg_macro>
         <xacro:leg_macro prefix="RRT" parent="RRF_link" type="fixed" mesh="rear_Toes_R.stl" color="orange">
             <axis xyz="1 0 0"/>
             <origin xyz="-0.003 0.088 0" rpy="0 0 0"/>
+            <box size="0.020 0.020 0.020"/>
         </xacro:leg_macro>
         <!-- === Rear left === -->
@@ -83,16 +96,20 @@
             <axis xyz="0 1 0"/>
             <origin xyz="0.027 0.04905 -0.00075" rpy="0 0 0"/>
+            <box size="0.032107 0.031304 0.01960"/>
         </xacro:leg_macro>
         <xacro:leg_macro prefix="RLL" parent="RLS_link" type="revolute" mesh="rear_Leg_L.stl" color="blue">
             <axis xyz="1 0 0"/>
             <origin xyz="0 0.022304 -0.01230" rpy="-1.57 0 0"/>
+            <box size="0.02905 0.07160 0.01960"/>
         </xacro:leg_macro>
         <xacro:leg_macro prefix="RLF" parent="RLL_link" type="revolute" mesh="rear_Foot_L.stl" color="purple">
             <axis xyz="1 0 0"/>
             <origin xyz="0.015546 0.054 0" rpy="0 0 0"/>
+            <box size="0.010 0.099465 0.010"/>
         </xacro:leg_macro>
         <xacro:leg_macro prefix="RLT" parent="RLF_link" type="fixed" mesh="rear_Toes_L.stl" color="orange">
             <axis xyz="1 0 0"/>
             <origin xyz="0.003 0.088 0" rpy="0 0 0"/>
+            <box size="0.020 0.020 0.020"/>
         </xacro:leg_macro>
     </robot>

File: quarobo_description/urdf/leg/leg.urdf.xacro (robot description, xacro)
@@ -2,5 +2,5 @@
 <robot xmlns:xacro="http://ros.org/wiki/xacro">
     <xacro:include filename="$(find quarobo_description)/urdf/material/material.urdf.xacro"/>
-    <xacro:macro name="leg_macro" params="prefix parent type mesh color *joint_axis *joint_origin">
+    <xacro:macro name="leg_macro" params="prefix parent type mesh color *joint_axis *joint_origin *collision_size">
         <joint name="${prefix}_joint" type="${type}">
             <parent link="${parent}"/>
@@ -13,5 +13,5 @@
             <inertial>
                 <origin xyz="0 0 0" rpy="0 0 0"/>
-                <mass value="0.02"/>
+                <mass value="0.020"/>
                 <inertia ixx="0.1" ixy="0" ixz="0" iyy="0.1" iyz="0" izz="0.1"/>
             </inertial>
@@ -26,5 +26,5 @@
                 <origin xyz="0 0 0" rpy="0 0 0"/>
                 <geometry>
-                    <xacro:insert_block name="link_box"/>
+                    <xacro:insert_block name="collision_size"/>
                 </geometry>
             </collision>
