Commit message: Add: quarobo_control directory; & Refactor;

File: quarobo_description/robots/quarobo.urdf.xacro (robot description, xacro)
@@ -3,129 +3,100 @@
     <xacro:include filename="$(find quarobo_description)/urdf/leg/leg.urdf.xacro"/>
     <link name="base_link"/>
-        <!-- === body === -->
-    <joint name="body_joint" type="fixed">
-        <parent link="base_link"/>
-        <child link="body_link"/>
+    <!-- === body === -->
+    <xacro:leg_macro_fi prefix="body" parent="base_link" mesh="body.stl" color="pink">
         <origin xyz="0 0 0.16505" rpy="0 0 0"/>
-    </joint>
-    <link name="body_link">
-        <inertial>
-            <origin xyz="0 0 0" rpy="0 0 0"/>
-            <mass value="0.020"/>
-            <inertia ixx="0.1" ixy="0" ixz="0" iyy="0.1" iyz="0" izz="0.1"/>
-        </inertial>
-        <visual>
-            <origin xyz="0 0 0" rpy="0 0 0"/>
-            <geometry>
-                <mesh filename="package://quarobo_description/meshes/origin_ros_quarobo_stlFiles/body.stl"/>
-            </geometry>
-            <material name="pink"/>
-        </visual>
-        <collision>
-            <origin xyz="0 0 0" rpy="0 0 0"/>
-            <geometry>
-                <box size="0.07160 0.09810 0.02410"/>
-            </geometry>
-        </collision>
-    </link>
+        <box size="0.07160 0.09810 0.02410"/>
+    </xacro:leg_macro_fi>
     <!-- === Front right === -->
-    <xacro:leg_macro prefix="FRS" parent="body_link" type="revolute" mesh="front_Shoulder_R.stl" color="green">
+    <xacro:leg_macro_re prefix="FRS" parent="body_link" mesh="front_Shoulder_R.stl" color="green">
         <origin xyz="-0.027 -0.04905 -0.00075" rpy="0 0 0"/>
         <axis xyz="0 1 0"/>
         <origin xyz="0 -0.010259 -0.002339" rpy="0 0 0"/>
         <box size="0.032107 0.031304 0.01960"/>
-    </xacro:leg_macro>
-    <xacro:leg_macro prefix="FRL" parent="FRS_link" type="revolute" mesh="front_Leg_R.stl" color="blue">
+    </xacro:leg_macro_re>
+    <xacro:leg_macro_re prefix="FRL" parent="FRS_link" mesh="front_Leg_R.stl" color="blue">
         <origin xyz="0 -0.022304 -0.01230" rpy="1.57 0 0"/>
         <axis xyz="1 0 0"/>
         <origin xyz="0 -0.02700 0" rpy="0 0 0"/>
         <box size="0.02905 0.07160 0.01960"/>
-    </xacro:leg_macro>
-    <xacro:leg_macro prefix="FRF" parent="FRL_link" type="revolute" mesh="front_Foot_R.stl" color="purple">
+    </xacro:leg_macro_re>
+    <xacro:leg_macro_re prefix="FRF" parent="FRL_link" mesh="front_Foot_R.stl" color="purple">
         <origin xyz="-0.015546 -0.054 0" rpy="0 0 0"/>
         <axis xyz="1 0 0"/>
         <origin xyz="-0.003069 -0.030498 0" rpy="0 0 0"/>
         <box size="0.010 0.099465 0.010"/>
-    </xacro:leg_macro>
-    <xacro:leg_macro prefix="FRT" parent="FRF_link" type="fixed" mesh="front_Toes_R.stl" color="orange">
+    </xacro:leg_macro_re>
+    <xacro:leg_macro_fi prefix="FRT" parent="FRF_link" mesh="front_Toes_R.stl" color="orange">
         <origin xyz="-0.003 -0.088 0" rpy="0 0 0"/>
-        <axis xyz="1 0 0"/>
-        <origin xyz="0 0 0" rpy="0 0 0"/>
         <box size="0.020 0.020 0.020"/>
-    </xacro:leg_macro>
+    </xacro:leg_macro_fi>
     <!-- === Front left === -->
-    <xacro:leg_macro prefix="FLS" parent="body_link" type="revolute" mesh="front_Shoulder_L.stl" color="green">
+    <xacro:leg_macro_re prefix="FLS" parent="body_link" mesh="front_Shoulder_L.stl" color="green">
         <origin xyz="0.027 -0.04905 -0.00075" rpy="0 0 0"/>
         <axis xyz="0 1 0"/>
         <origin xyz="0 -0.010259 -0.002339" rpy="0 0 0"/>
         <box size="0.032107 0.031304 0.01960"/>
-    </xacro:leg_macro>
-    <xacro:leg_macro prefix="FLL" parent="FLS_link" type="revolute" mesh="front_Leg_L.stl" color="blue">
+    </xacro:leg_macro_re>
+    <xacro:leg_macro_re prefix="FLL" parent="FLS_link" mesh="front_Leg_L.stl" color="blue">
         <origin xyz="0 -0.022304 -0.01230" rpy="1.57 0 0"/>
         <axis xyz="1 0 0"/>
         <origin xyz="0 -0.02700 0" rpy="0 0 0"/>
         <box size="0.02905 0.07160 0.01960"/>
-    </xacro:leg_macro>
-    <xacro:leg_macro prefix="FLF" parent="FLL_link" type="revolute" mesh="front_Foot_L.stl" color="purple">
+    </xacro:leg_macro_re>
+    <xacro:leg_macro_re prefix="FLF" parent="FLL_link" mesh="front_Foot_L.stl" color="purple">
         <origin xyz="0.015546 -0.054 0" rpy="0 0 0"/>
         <axis xyz="1 0 0"/>
         <origin xyz="0.003069 -0.030498 0" rpy="0 0 0"/>
         <box size="0.010 0.099465 0.010"/>
-    </xacro:leg_macro>
-    <xacro:leg_macro prefix="FLT" parent="FLF_link" type="fixed" mesh="front_Toes_L.stl" color="orange">
+    </xacro:leg_macro_re>
+    <xacro:leg_macro_fi prefix="FLT" parent="FLF_link" mesh="front_Toes_L.stl" color="orange">
         <origin xyz="0.003 -0.088 0" rpy="0 0 0"/>
-        <axis xyz="1 0 0"/>
-        <origin xyz="0 0 0" rpy="0 0 0"/>
         <box size="0.020 0.020 0.020"/>
-    </xacro:leg_macro>
+    </xacro:leg_macro_fi>
     <!-- === Rear right === -->
-    <xacro:leg_macro prefix="RRS" parent="body_link" type="revolute" mesh="rear_Shoulder_R.stl" color="green">
+    <xacro:leg_macro_re prefix="RRS" parent="body_link" mesh="rear_Shoulder_R.stl" color="green">
         <origin xyz="-0.027 0.04905 -0.00075" rpy="0 0 0"/>
         <axis xyz="0 1 0"/>
         <origin xyz="0 0.010259 -0.002339" rpy="0 0 0"/>
         <box size="0.032107 0.031304 0.01960"/>
-    </xacro:leg_macro>
-    <xacro:leg_macro prefix="RRL" parent="RRS_link" type="revolute" mesh="rear_Leg_R.stl" color="blue">
+    </xacro:leg_macro_re>
+    <xacro:leg_macro_re prefix="RRL" parent="RRS_link" mesh="rear_Leg_R.stl" color="blue">
         <origin xyz="0 0.022304 -0.01230" rpy="-1.57 0 0"/>
         <axis xyz="1 0 0"/>
         <origin xyz="0 0.02700 0" rpy="0 0 0"/>
         <box size="0.02905 0.07160 0.01960"/>
-    </xacro:leg_macro>
-    <xacro:leg_macro prefix="RRF" parent="RRL_link" type="revolute" mesh="rear_Foot_R.stl" color="purple">
+    </xacro:leg_macro_re>
+    <xacro:leg_macro_re prefix="RRF" parent="RRL_link" mesh="rear_Foot_R.stl" color="purple">
         <origin xyz="-0.015546 0.054 0" rpy="0 0 0"/>
         <axis xyz="1 0 0"/>
         <origin xyz="-0.003069 0.030498 0" rpy="0 0 0"/>
         <box size="0.010 0.099465 0.010"/>
-    </xacro:leg_macro>
-    <xacro:leg_macro prefix="RRT" parent="RRF_link" type="fixed" mesh="rear_Toes_R.stl" color="orange">
+    </xacro:leg_macro_re>
+    <xacro:leg_macro_fi prefix="RRT" parent="RRF_link" mesh="rear_Toes_R.stl" color="orange">
         <origin xyz="-0.003 0.088 0" rpy="0 0 0"/>
-        <axis xyz="1 0 0"/>
-        <origin xyz="0 0 0" rpy="0 0 0"/>
         <box size="0.020 0.020 0.020"/>
-    </xacro:leg_macro>
+    </xacro:leg_macro_fi>
     <!-- === Rear left === -->
-    <xacro:leg_macro prefix="RLS" parent="body_link" type="revolute" mesh="rear_Shoulder_L.stl" color="green">
+    <xacro:leg_macro_re prefix="RLS" parent="body_link" mesh="rear_Shoulder_L.stl" color="green">
         <origin xyz="0.027 0.04905 -0.00075" rpy="0 0 0"/>
         <axis xyz="0 1 0"/>
         <origin xyz="0 0.010259 -0.002339" rpy="0 0 0"/>
         <box size="0.032107 0.031304 0.01960"/>
-    </xacro:leg_macro>
-    <xacro:leg_macro prefix="RLL" parent="RLS_link" type="revolute" mesh="rear_Leg_L.stl" color="blue">
+    </xacro:leg_macro_re>
+    <xacro:leg_macro_re prefix="RLL" parent="RLS_link" mesh="rear_Leg_L.stl" color="blue">
         <origin xyz="0 0.022304 -0.01230" rpy="-1.57 0 0"/>
         <axis xyz="1 0 0"/>
         <origin xyz="0 0.02700 0" rpy="0 0 0"/>
         <box size="0.02905 0.07160 0.01960"/>
-    </xacro:leg_macro>
-    <xacro:leg_macro prefix="RLF" parent="RLL_link" type="revolute" mesh="rear_Foot_L.stl" color="purple">
+    </xacro:leg_macro_re>
+    <xacro:leg_macro_re prefix="RLF" parent="RLL_link" mesh="rear_Foot_L.stl" color="purple">
         <origin xyz="0.015546 0.054 0" rpy="0 0 0"/>
         <axis xyz="1 0 0"/>
         <origin xyz="0.003069 0.030498 0" rpy="0 0 0"/>
         <box size="0.010 0.099465 0.010"/>
-    </xacro:leg_macro>
-    <xacro:leg_macro prefix="RLT" parent="RLF_link" type="fixed" mesh="rear_Toes_L.stl" color="orange">
+    </xacro:leg_macro_re>
+    <xacro:leg_macro_fi prefix="RLT" parent="RLF_link" mesh="rear_Toes_L.stl" color="orange">
         <origin xyz="0.003 0.088 0" rpy="0 0 0"/>
-        <axis xyz="1 0 0"/>
-        <origin xyz="0 0 0" rpy="0 0 0"/>
         <box size="0.020 0.020 0.020"/>
-    </xacro:leg_macro>
+    </xacro:leg_macro_fi>
 </robot>

File: quarobo_description/urdf/leg/leg.urdf.xacro (robot description, xacro)
@@ -2,6 +2,38 @@
 <robot xmlns:xacro="http://ros.org/wiki/xacro">
     <xacro:include filename="$(find quarobo_description)/urdf/material/material.urdf.xacro"/>
-    <xacro:macro name="leg_macro" params="prefix parent type mesh color *joint_origin *joint_axis *collision_origin *collision_size">
-        <joint name="${prefix}_joint" type="${type}">
+        <!-- === fixed === -->
+    <xacro:macro name="leg_macro_fi" params="prefix parent mesh color *joint_origin *collision_size">
+        <joint name="${prefix}_joint" type="fixed">
+            <parent link="${parent}"/>
+            <child link="${prefix}_link"/>
+            <xacro:insert_block name="joint_origin"/>
+        </joint>
+        <link name="${prefix}_link">
+            <inertial>
+                <origin xyz="0 0 0" rpy="0 0 0"/>
+                <mass value="0.020"/>
+                <inertia
+                    ixx="0.1" ixy="0" ixz="0"
+                    iyy="0.1" iyz="0"
+                    izz="0.1"/>
+            </inertial>
+            <visual>
+                <origin xyz="0 0 0" rpy="0 0 0"/>
+                <geometry>
+                    <mesh filename="package://quarobo_description/meshes/origin_ros_quarobo_stlFiles/${mesh}"/>
+                </geometry>
+                <material name="${color}"/>
+            </visual>
+            <collision>
+                <origin xyz="0 0 0" rpy="0 0 0"/>
+                <geometry>
+                    <xacro:insert_block name="collision_size"/>
+                </geometry>
+            </collision>
+        </link>
+    </xacro:macro>
+    <!-- === revolute === -->
+    <xacro:macro name="leg_macro_re" params="prefix parent mesh color *joint_origin *joint_axis *collision_origin *collision_size">
+        <joint name="${prefix}_joint" type="revolute">
             <parent link="${parent}"/>
             <child link="${prefix}_link"/>
@@ -9,4 +41,5 @@
             <xacro:insert_block name="joint_axis"/>
             <limit lower="-2.61" upper="2.61" effort="1000" velocity="0.5"/>
+            <dynamics damping="0.1"/>
         </joint>
         <link name="${prefix}_link">
@@ -14,5 +47,8 @@
                 <origin xyz="0 0 0" rpy="0 0 0"/>
                 <mass value="0.020"/>
-                <inertia ixx="0.1" ixy="0" ixz="0" iyy="0.1" iyz="0" izz="0.1"/>
+                <inertia
+                    ixx="0.1" ixy="0" ixz="0"
+                    iyy="0.1" iyz="0"
+                    izz="0.1"/>
             </inertial>
             <visual>
