Commit message: Commit for now.

File: quarobo_description/robots/old_quarobo.urdf.xacro (robot description, xacro)
@@ -6,4 +6,5 @@
     <xacro:leg_macro_fi prefix="body" parent="base_link" mesh="body.stl" color="pink">
         <origin xyz="0 0 0.16505" rpy="0 0 0"/>
+        <box size="0.07160 0.09810 0.02410"/>
     </xacro:leg_macro_fi>
     <!-- === Front right === -->
@@ -11,15 +12,22 @@
         <origin xyz="-0.027 -0.04905 -0.00075" rpy="0 0 0"/>
         <axis xyz="0 1 0"/>
+        <origin xyz="0 -0.010259 -0.002339" rpy="0 0 0"/>
+        <box size="0.032107 0.031304 0.01960"/>
     </xacro:leg_macro_re>
     <xacro:leg_macro_re prefix="FRL" parent="FRS_link" mesh="front_Leg_R.stl" color="blue">
         <origin xyz="0 -0.022304 -0.01230" rpy="1.57 0 0"/>
         <axis xyz="1 0 0"/>
+        <origin xyz="0 -0.02700 0" rpy="0 0 0"/>
+        <box size="0.02905 0.07160 0.01960"/>
     </xacro:leg_macro_re>
     <xacro:leg_macro_re prefix="FRF" parent="FRL_link" mesh="front_Foot_R.stl" color="purple">
         <origin xyz="-0.015546 -0.054 0" rpy="0 0 0"/>
         <axis xyz="1 0 0"/>
+        <origin xyz="-0.003069 -0.030498 0" rpy="0 0 0"/>
+        <box size="0.010 0.099465 0.010"/>
     </xacro:leg_macro_re>
     <xacro:leg_macro_fi prefix="FRT" parent="FRF_link" mesh="front_Toes_R.stl" color="orange">
         <origin xyz="-0.003 -0.088 0" rpy="0 0 0"/>
+        <box size="0.020 0.020 0.020"/>
     </xacro:leg_macro_fi>
     <!-- === Front left === -->
@@ -27,15 +35,22 @@
         <origin xyz="0.027 -0.04905 -0.00075" rpy="0 0 0"/>
         <axis xyz="0 1 0"/>
+        <origin xyz="0 -0.010259 -0.002339" rpy="0 0 0"/>
+        <box size="0.032107 0.031304 0.01960"/>
     </xacro:leg_macro_re>
     <xacro:leg_macro_re prefix="FLL" parent="FLS_link" mesh="front_Leg_L.stl" color="blue">
         <origin xyz="0 -0.022304 -0.01230" rpy="1.57 0 0"/>
         <axis xyz="1 0 0"/>
+        <origin xyz="0 -0.02700 0" rpy="0 0 0"/>
+        <box size="0.02905 0.07160 0.01960"/>
     </xacro:leg_macro_re>
     <xacro:leg_macro_re prefix="FLF" parent="FLL_link" mesh="front_Foot_L.stl" color="purple">
         <origin xyz="0.015546 -0.054 0" rpy="0 0 0"/>
         <axis xyz="1 0 0"/>
+        <origin xyz="0.003069 -0.030498 0" rpy="0 0 0"/>
+        <box size="0.010 0.099465 0.010"/>
     </xacro:leg_macro_re>
     <xacro:leg_macro_fi prefix="FLT" parent="FLF_link" mesh="front_Toes_L.stl" color="orange">
         <origin xyz="0.003 -0.088 0" rpy="0 0 0"/>
+        <box size="0.020 0.020 0.020"/>
     </xacro:leg_macro_fi>
     <!-- === Rear right === -->
@@ -43,15 +58,22 @@
         <origin xyz="-0.027 0.04905 -0.00075" rpy="0 0 0"/>
         <axis xyz="0 1 0"/>
+        <origin xyz="0 0.010259 -0.002339" rpy="0 0 0"/>
+        <box size="0.032107 0.031304 0.01960"/>
     </xacro:leg_macro_re>
     <xacro:leg_macro_re prefix="RRL" parent="RRS_link" mesh="rear_Leg_R.stl" color="blue">
         <origin xyz="0 0.022304 -0.01230" rpy="-1.57 0 0"/>
         <axis xyz="1 0 0"/>
+        <origin xyz="0 0.02700 0" rpy="0 0 0"/>
+        <box size="0.02905 0.07160 0.01960"/>
     </xacro:leg_macro_re>
     <xacro:leg_macro_re prefix="RRF" parent="RRL_link" mesh="rear_Foot_R.stl" color="purple">
         <origin xyz="-0.015546 0.054 0" rpy="0 0 0"/>
         <axis xyz="1 0 0"/>
+        <origin xyz="-0.003069 0.030498 0" rpy="0 0 0"/>
+        <box size="0.010 0.099465 0.010"/>
     </xacro:leg_macro_re>
     <xacro:leg_macro_fi prefix="RRT" parent="RRF_link" mesh="rear_Toes_R.stl" color="orange">
         <origin xyz="-0.003 0.088 0" rpy="0 0 0"/>
+        <box size="0.020 0.020 0.020"/>
     </xacro:leg_macro_fi>
     <!-- === Rear left === -->
@@ -59,15 +81,22 @@
         <origin xyz="0.027 0.04905 -0.00075" rpy="0 0 0"/>
         <axis xyz="0 1 0"/>
+        <origin xyz="0 0.010259 -0.002339" rpy="0 0 0"/>
+        <box size="0.032107 0.031304 0.01960"/>
     </xacro:leg_macro_re>
     <xacro:leg_macro_re prefix="RLL" parent="RLS_link" mesh="rear_Leg_L.stl" color="blue">
         <origin xyz="0 0.022304 -0.01230" rpy="-1.57 0 0"/>
         <axis xyz="1 0 0"/>
+        <origin xyz="0 0.02700 0" rpy="0 0 0"/>
+        <box size="0.02905 0.07160 0.01960"/>
     </xacro:leg_macro_re>
     <xacro:leg_macro_re prefix="RLF" parent="RLL_link" mesh="rear_Foot_L.stl" color="purple">
         <origin xyz="0.015546 0.054 0" rpy="0 0 0"/>
         <axis xyz="1 0 0"/>
+        <origin xyz="0.003069 0.030498 0" rpy="0 0 0"/>
+        <box size="0.010 0.099465 0.010"/>
     </xacro:leg_macro_re>
     <xacro:leg_macro_fi prefix="RLT" parent="RLF_link" mesh="rear_Toes_L.stl" color="orange">
         <origin xyz="0.003 0.088 0" rpy="0 0 0"/>
+        <box size="0.020 0.020 0.020"/>
     </xacro:leg_macro_fi>
 </robot>

File: quarobo_description/urdf/leg/old_leg.urdf.xacro (robot description, xacro)
@@ -3,5 +3,5 @@
     <xacro:include filename="$(find quarobo_description)/urdf/material/material.urdf.xacro"/>
         <!-- === fixed === -->
-    <xacro:macro name="leg_macro_fi" params="prefix parent mesh color *joint_origin">
+    <xacro:macro name="leg_macro_fi" params="prefix parent mesh color *joint_origin *collision_size">
         <joint name="${prefix}_joint" type="fixed">
             <parent link="${parent}"/>
@@ -25,8 +25,14 @@
                 <material name="${color}"/>
             </visual>
+            <collision>
+                <origin xyz="0 0 0" rpy="0 0 0"/>
+                <geometry>
+                    <xacro:insert_block name="collision_size"/>
+                </geometry>
+            </collision>
         </link>
     </xacro:macro>
     <!-- === revolute === -->
-    <xacro:macro name="leg_macro_re" params="prefix parent mesh color *joint_origin *joint_axis">
+    <xacro:macro name="leg_macro_re" params="prefix parent mesh color *joint_origin *joint_axis *collision_origin *collision_size">
         <joint name="${prefix}_joint" type="revolute">
             <parent link="${parent}"/>
@@ -53,4 +59,10 @@
                 <material name="${color}"/>
             </visual>
+            <collision>
+                <xacro:insert_block name="collision_origin"/>
+                <geometry>
+                    <xacro:insert_block name="collision_size"/>
+                </geometry>
+            </collision>
         </link>
     </xacro:macro>
